Commit message: arm_controller adapted to UR, made a lot of hacks, will need work to be legit

File: ur_arm/ur_description/urdf/ur.urdf.xacro (robot description, xacro)
@@ -26,18 +26,4 @@
      <kd>1.0</kd>
   </xacro:macro>
-    <!-- IMPORTANT NOTE about arm and finger limits: These values are optimized for mass dividers between 2 (for fingers 1-3)
-         for using gazebo_ros_control hardware interface controllers.
-         The seemingly most important factor in making robots explode is too much force allowed. Higher PID gains don't have too
-         much of an effect. Should maybe start testing with higher PID values to challenge hitting the max force.
-         The mass also plays a role. The lighter the robot, the easier it explodes when movements are made.
-         When it is heavy, it is harder to lift the arm, and when it moves down, there's a risk of it collapsing down and then exploding after.
-         For fingers: with current values, it works only with starting from 1.1 - 1.0 doesn't move. When it's too high, the robot explodes (last tested with finger mass div 1).
-         Velocity was tested between 0.1 and 0.3 but not sure it has an effect.
-         UPDATE 30.1: reducing the damping and friction for some joints has greatly improved the outcome. Damping/Friction probably also has played a roll in the robot collapses. -->
-  <!-- Note for reading this in gazebo model (2015): effort and velocity limits are not yet imported properly in gazebo.
-         Update the driver after it does! Now it's hard-coded in C Macros -->
-  <xacro:macro name="default_finger_limits">
-    <limit lower="-0.0045" upper="1.05" effort="1.5" velocity="0.2" />
-  </xacro:macro>
   <xacro:macro name="arm_0_limits">
     <limit effort="8" velocity="1.0" />
@@ -67,11 +53,4 @@
   <xacro:macro name="default_damping_high">
     <dynamics damping="0.7" friction="1.0"/>
-  </xacro:macro>
-  <xacro:macro name="damping_fingers">
-    <!--- remark 2014: damping greater than 0.1 (0.2) lead to model break downs when testing it bit by bit -->
-        <!--- remark jan 2016: damping and friction higher than 0.005 required very high forces in order for the fingers
-              to move at all, and then they mooved only slowly. -->
-    <!--dynamics damping="0.1" friction="1.0"/-->
-    <dynamics damping="0.005" friction="0.005"/>
   </xacro:macro>
   <!-- Formula according to https://en.wikipedia.org/wiki/List_of_moment_of_inertia_tensors for cylinder -->
@@ -107,7 +86,7 @@
   <!-- ***************** MODEL CORRECTIONS ************************* -->
   <!-- MODEL_FIX corrections for hand limb, which is not modelled correctly.
-  <xacro:property name="wrist_scale_x" value="1.12"/>
-  <xacro:property name="wrist_scale_y" value="1.05"/>
-  <xacro:property name="wrist_scale_z" value="1.05"/>
+  <xacro:property name="wrist_scale_x" value="1.0"/>
+  <xacro:property name="wrist_scale_y" value="1.0"/>
+  <xacro:property name="wrist_scale_z" value="1.0"/>
   -->
   <xacro:property name="wrist_scale_x" value="1.0"/>
@@ -115,42 +94,9 @@
   <xacro:property name="wrist_scale_z" value="1.0"/>
   <!-- MODEL_FIX transform of base to first joint as derived from DH specs is not exact, this is a correction
-  <xacro:property name="base_height_corr" value="-0.005"/>
-  <xacro:property name="base_height_corr" value="-0.005"/>
+  <xacro:property name="base_height_corr" value="0"/>
+  <xacro:property name="base_height_corr" value="0"/>
 -->
   <xacro:property name="base_height_corr" value="0"/>
   <xacro:property name="base_height_corr" value="0"/>
-  <!-- MODEL_FIX finger tip visuals are not long enough -->
-  <!--
-  <xacro:property name="tip_scale_x" value="1.17"/>
-  <xacro:property name="tip_scale_y" value="1"/>
-  <xacro:property name="tip_scale_z" value="1"/>
-  -->
-  <xacro:property name="tip_scale_x" value="1"/>
-  <xacro:property name="tip_scale_y" value="1"/>
-  <xacro:property name="tip_scale_z" value="1"/>
-  <!-- *************************************************************** -->
-  <!-- MODEL_FIX transforms from wrist to finger joints. Measures from the kinova spec image (Hand.png), pitch angles calculated from measures and experimentally adapted -->
-  <!--<xacro:property name="f_thb_xyz" value=" 0.0319  0.003  0.1214" />
-  <xacro:property name="f_idx_xyz" value="-0.0276  0.0204 0.1214" />
-  <xacro:property name="f_pnk_xyz" value="-0.0276 -0.0204 0.1214" /> -->
-  <xacro:property name="f_thb_xyz" value=" 0.0319  0.003  0.11" />
-  <xacro:property name="f_idx_xyz" value="-0.0276  0.0204 0.11" />
-  <xacro:property name="f_pnk_xyz" value="-0.0276 -0.0204 0.11" />
-  <xacro:property name="f_thb_rpy" value="0 -0.37 ${M_PI-0.226892}" /> <!-- from measurements, pitch is -0.2658 -->
-  <xacro:property name="f_idx_rpy" value="0 -0.34 -0.191986" /> <!-- from measurements, pitch is -0.2293 -->
-  <xacro:property name="f_pnk_rpy" value="0 -0.34 0.191986" /> <!-- from measurements, pitch is -0.2293 -->
-  <!-- MODEL_FIX transforms from wrist to finger mounts -->
-  <!--<xacro:property name="f_thb_m_xyz" value=" 0.037  0.001  0.106" />
-  <xacro:property name="f_idx_m_xyz" value="-0.034  0.022 0.106" />
-  <xacro:property name="f_pnk_m_xyz" value="-0.034 -0.022 0.106" />
-  <xacro:property name="f_thb_m_rpy" value="0 -0.2658 ${M_PI-0.226892}" />
-  <xacro:property name="f_idx_m_rpy" value="0 -0.2293 -0.191986" />
-  <xacro:property name="f_pnk_m_rpy" value="0 -0.2293 0.191986" />-->
-  <xacro:property name="f_thb_m_xyz" value=" 0.037  0.001  0.095" />
-  <xacro:property name="f_idx_m_xyz" value="-0.034  0.022 0.095" />
-  <xacro:property name="f_pnk_m_xyz" value="-0.034 -0.022 0.095" />
-  <xacro:property name="f_thb_m_rpy" value="0 -0.2658 ${M_PI-0.226892}" />
-  <xacro:property name="f_idx_m_rpy" value="0 -0.2293 -0.191986" />
-  <xacro:property name="f_pnk_m_rpy" value="0 -0.2293 0.191986" />
   <!-- MACRO FOR THE ROBOT ARM -->
   <xacro:macro name="ur_arm" params="parent mass_divider finger_mass_divider *origin ur_prefix:=ur">
@@ -172,9 +118,4 @@
     <xacro:default_material/>
   </gazebo>
-  <gazebo reference="_finger">
-    <material>Gazebo/Grey</material>
-    <implicitSpringDamper>1</implicitSpringDamper>
-    <xacro:default_material/>
-  </gazebo>
   <!-- for some reason, material only applies if full name specified -->
   <gazebo reference="${ur_prefix}base">
@@ -205,4 +146,13 @@
     <material>Gazebo/FlatBlack</material>
     <xacro:default_material/>
+  </gazebo>
+  <gazebo reference="${ur_prefix}_finger_joint_0">
+    <provideFeedback value="true"/>
+  </gazebo>
+    <gazebo reference="${ur_prefix}_finger_joint_2">
+    <provideFeedback value="true"/>
+  </gazebo>
+    <gazebo reference="${ur_prefix}_finger_joint_4">
+    <provideFeedback value="true"/>
   </gazebo>
     <xacro:if value="$(arg add_transmission_pos)">
@@ -214,13 +164,78 @@
         <xacro:ur_joint_control_vel ur_prefix="${ur_prefix}"/>
     </xacro:if>
+  <xacro:property name="pi" value="3.14159265" />
+  <!-- Inertia parameters -->
+  <xacro:property name="base_mass" value="4.0" />  <!-- This mass might be incorrect -->
+  <xacro:property name="shoulder_mass" value="3.7000" />
+  <xacro:property name="upper_arm_mass" value="8.3930" />
+  <xacro:property name="forearm_mass" value="2.2750" />
+  <xacro:property name="wrist_1_mass" value="1.2190" />
+  <xacro:property name="wrist_2_mass" value="1.2190" />
+  <xacro:property name="wrist_3_mass" value="0.1879" />
+  <xacro:property name="shoulder_cog" value="0.0 0.00193 -0.02561" />
+  <xacro:property name="upper_arm_cog" value="0.0 -0.024201 0.2125" />
+  <xacro:property name="forearm_cog" value="0.0 0.0265 0.11993" />
+  <xacro:property name="wrist_1_cog" value="0.0 0.110949 0.01634" />
+  <xacro:property name="wrist_2_cog" value="0.0 0.0018 0.11099" />
+  <xacro:property name="wrist_3_cog" value="0.0 0.001159 0.0" />
+  <!-- Kinematic model -->
+  <!-- Properties from urcontrol.conf -->
+  <!--
+    DH for UR5:
+    a = [0.00000, -0.42500, -0.39225,  0.00000,  0.00000,  0.0000]
+    d = [0.089159,  0.00000,  0.00000,  0.10915,  0.09465,  0.0823]
+    alpha = [ 1.570796327, 0, 0, 1.570796327, -1.570796327, 0 ]
+    q_home_offset = [0, -1.570796327, 0, -1.570796327, 0, 0]
+    joint_direction = [-1, -1, 1, 1, 1, 1]
+    mass = [3.7000, 8.3930, 2.2750, 1.2190, 1.2190, 0.1879]
+    center_of_mass = [ [0, -0.02561, 0.00193], [0.2125, 0, 0.11336], [0.11993, 0.0, 0.0265], [0, -0.0018, 0.01634], [0, 0.0018,0.01634], [0, 0, -0.001159] ]
+  -->
+  <xacro:property name="ur_d1" value="0.089159" />
+  <xacro:property name="ur_a2" value="-0.42500" />
+  <xacro:property name="ur_a3" value="-0.39225" />
+  <xacro:property name="ur_d4" value="0.10915" />
+  <xacro:property name="ur_d5" value="0.09465" />
+  <xacro:property name="ur_d6" value="0.0823" />
+  <!-- Arbitrary offsets for shoulder/elbow joints -->
+  <xacro:property name="shoulder_offset" value="0.13585" />  <!-- measured from model -->
+  <xacro:property name="elbow_offset" value="-0.1197" /> <!-- measured from model -->
+  <!-- link lengths used in model -->
+  <xacro:property name="shoulder_height" value="${ur_d1}" />
+  <xacro:property name="upper_arm_length" value="${-ur_a2}" />
+  <xacro:property name="forearm_length" value="${-ur_a3}" />
+  <xacro:property name="wrist_1_length" value="${ur_d4 - elbow_offset - shoulder_offset}" />
+  <xacro:property name="wrist_2_length" value="${ur_d5}" />
+  <xacro:property name="wrist_3_length" value="${ur_d6}" />
+  <!--property name="shoulder_height" value="0.089159" /-->
+  <!--property name="shoulder_offset" value="0.13585" /-->  <!-- shoulder_offset - elbow_offset + wrist_1_length = 0.10915 -->
+  <!--property name="upper_arm_length" value="0.42500" /-->
+  <!--property name="elbow_offset" value="0.1197" /-->       <!-- CAD measured -->
+  <!--property name="forearm_length" value="0.39225" /-->
+  <!--property name="wrist_1_length" value="0.093" /-->     <!-- CAD measured -->
+  <!--property name="wrist_2_length" value="0.09465" /-->   <!-- In CAD this distance is 0.930, but in the spec it is 0.09465 -->
+  <!--property name="wrist_3_length" value="0.0823" /-->
+  <xacro:property name="shoulder_radius" value="0.060" />   <!-- manually measured -->
+  <xacro:property name="upper_arm_radius" value="0.054" />  <!-- manually measured -->
+  <xacro:property name="elbow_radius" value="0.060" />      <!-- manually measured -->
+  <xacro:property name="forearm_radius" value="0.040" />    <!-- manually measured -->
+  <xacro:property name="wrist_radius" value="0.045" />      <!-- manually measured -->
+  <xacro:macro name="cylinder_inertial" params="radius length mass *origin">
+    <inertial>
+      <mass value="${mass}" />
+      <xacro:insert_block name="origin" />
+      <inertia ixx="${0.0833333 * mass * (3 * radius * radius + length * length)}" ixy="0.0" ixz="0.0"
+        iyy="${0.0833333 * mass * (3 * radius * radius + length * length)}" iyz="0.0"
+        izz="${0.5 * mass * radius * radius}" />
+    </inertial>
+  </xacro:macro>
   <link name="${ur_prefix}_0_baseA">
     <inertial>
-      <origin xyz="0 0 0.03" rpy="0 0 0" />
-      <xacro:cyl_inertia mass="${0.5688/mass_divider}" h="0.059" r="0.036"/>
+      <origin xyz="0 0 0.0" rpy="0 0 0" />
+      <xacro:cyl_inertia mass="${0.5688}" h="0.059" r="0.036"/>
     </inertial>
     <visual>
       <origin xyz="0 0 0" rpy="0 0 0" />
       <geometry>
-        <mesh filename="package://ur_description/meshes/ur2/0_baseA.STL"  scale="0.98 0.98 0.98"/>
+        <mesh filename="package://ur_description/meshes/ur/base.stl"/>
       </geometry>
       <material name="">
@@ -231,671 +246,297 @@
       <origin xyz="0 0 0" rpy="0 0 0" />
       <geometry>
-        <mesh filename="package://ur_description/meshes/ur2/0_baseA.STL" />
+        <mesh filename="package://ur_description/meshes/ur/base.stl"/>
       </geometry>
     </collision>
   </link>
-  <!-- ...........................        -->
-  <link name="${ur_prefix}_0_baseB_limb">
+   <link name="${ur_prefix}_0_baseB_limb">
     <inertial>
-      <origin xyz="0 0.04725 0" rpy="0 0 0" />
-      <xacro:cyl_inertia mass="${0.5152/mass_divider}" h="0.0945" r="0.04"/>
+      <origin xyz="0 0 0.0" rpy="0 0 0" />
+      <xacro:cyl_inertia mass="${0.5688}" h="0.059" r="0.036"/>
     </inertial>
     <visual>
       <origin xyz="0 0 0" rpy="0 0 0" />
       <geometry>
-        <mesh filename="package://ur_description/meshes/ur2/0_baseB_limb.STL"/>
+        <mesh filename="package://ur_description/meshes/ur/base.stl"/>
       </geometry>
-      <material name="">
-        <color rgba="0.10 0.10 0.10 1" />
-      </material>
+        <material name="LightGrey">
+          <color rgba="0.7 0.7 0.7 1.0"/>
+        </material>
     </visual>
     <collision>
       <origin xyz="0 0 0" rpy="0 0 0" />
       <geometry>
-        <mesh filename="package://ur_description/meshes/ur2/0_baseB_limb.STL" />
+        <mesh filename="package://ur_description/meshes/ur/base.stl" />
       </geometry>
     </collision>
   </link>
     <joint name="${ur_prefix}_base_internal" type="fixed">
-    <origin xyz="0 0 ${0.049 + base_height_corr}" rpy="${M_PI_2} 0 0" />
+    <origin xyz="0 0 0" rpy="0 0 0" />
         <parent link="${ur_prefix}_0_baseA" />
         <child link="${ur_prefix}_0_baseB_limb" />
     <axis xyz="0 0 0" />
   </joint>
-  <link name="${ur_prefix}_ring_1">
-    <inertial>
-      <origin xyz="-3.57503886452221E-16 -1.58125151997128E-15 -5.55111512312578E-17" rpy="0 0 0" />
-      <xacro:cyl_inertia mass="${0.00872/mass_divider}" h="0.02" r="0.04"/>
-    </inertial>
-    <visual>
-      <origin xyz="0 0 0" rpy="0 0 0" />
-      <geometry>
-        <mesh filename="package://ur_description/meshes/ur2/ring_1.STL" />
-      </geometry>
-      <material name="">
-        <color rgba="0.50 0.50 0.50 1" />
-      </material>
-    </visual>
-    <collision>
-      <origin xyz="0 0 0" rpy="0 0 0" />
-      <geometry>
-        <mesh filename="package://ur_description/meshes/ur2/ring_1.STL" />
-      </geometry>
-    </collision>
-  </link>
-    <joint name="${ur_prefix}_ring_1_joint" type="fixed">
-    <origin xyz="0 0.104 0" rpy="-${M_PI_2} 0.211499083190217 -${M_PI}" />
-        <parent link="${ur_prefix}_0_baseB_limb" />
-        <child link="${ur_prefix}_ring_1" />
-    <axis xyz="0 0 0" />
-  </joint>
-  <!-- ...........................        -->
-  <link name="${ur_prefix}_1_shoulder_limb">
-    <inertial>
-      <origin xyz="0.0120470281905243 0.0657132437750733 0" rpy="0 0 0" />
-      <xacro:cyl_inertia mass="${0.4782/mass_divider}" h="0.159" r="0.04"/>
-    </inertial>
-    <visual>
-      <origin xyz="0 0 0" rpy="0 0 0" />
-      <geometry>
-        <mesh filename="package://ur_description/meshes/ur2/1_shoulder_limb.STL" />
-      </geometry>
-      <material name="">
-        <color rgba="0.10 0.10 0.10 1" />
-      </material>
-    </visual>
-    <xacro:testSphere/>
-    <collision>
-      <origin xyz="0 0 0" rpy="0 0 0" />
-      <geometry>
-        <mesh filename="package://ur_description/meshes/ur2/1_shoulder_limb.STL" />
-      </geometry>
-    </collision>
-  </link>
-    <joint name="${ur_prefix}_arm_0_joint" type="continuous">
-    <xacro:arm_0_limits/>
-     <xacro:default_damping_medium/>
-    <origin xyz="0 0.104 0" rpy="0 ${M_PI_2} 0" />
-        <parent link="${ur_prefix}_0_baseB_limb" />
-        <child link="${ur_prefix}_1_shoulder_limb" />
-    <axis xyz="0 1 0" />
-  </joint>
-  <!-- ...........................        -->
-    <link name="${ur_prefix}_ring_2">
-    <inertial>
-      <origin xyz="0 0 0" rpy="0 0 0" />
-      <xacro:cyl_inertia mass="${0.00872/mass_divider}" h="0.02" r="0.04"/>
-    </inertial>
-    <visual>
-      <origin xyz="-0.0005 -0.003 -0.001" rpy="0 0 0" />
-      <geometry>
-        <mesh filename="package://ur_description/meshes/ur2/ring_2.STL" />
-      </geometry>
-      <material name="">
-        <color rgba="0.50 0.50 0.50 1" />
-      </material>
-    </visual>
-    <collision>
-      <origin xyz="-0.0005 -0.003 -0.001" rpy="0 0 0" />
-      <geometry>
-        <mesh filename="package://ur_description/meshes/ur2/ring_2.STL" />
-      </geometry>
-    </collision>
-  </link>
-    <joint name="${ur_prefix}_ring_2_joint" type="fixed">
-    <origin xyz="0 0.1225 0" rpy="-1.57079632679488 -1.49007956532211 1.57079632679488" />
-        <parent link="${ur_prefix}_1_shoulder_limb" />
-        <child link="${ur_prefix}_ring_2" />
-    <axis xyz="0 0 0" />
-  </joint>
-  <!-- ...........................        -->
-  <link name="${ur_prefix}_2_upperarm_limb">
-    <inertial>
-      <origin xyz="0.206003857152394 0 -0.0343672381612413" rpy="0 0 0" />
-      <xacro:cyl_inertia mass="${1.37163/mass_divider}" h="0.49" r="0.049"/>
-    </inertial>
-    <visual>
-      <origin xyz="-0.003 -0.001 -0.001" rpy="0 0 0" />
-      <geometry>
-        <mesh filename="package://ur_description/meshes/ur2/2_upperarm_limb.STL" />
-      </geometry>
-      <material name="">
-        <color rgba="0.10 0.10 0.10 1" />
-      </material>
-    </visual>
-     <xacro:testSphere/>
-    <collision>
-      <origin xyz="-0.003 -0.001 -0.001" rpy="0 0 0" />
-      <geometry>
-        <mesh filename="package://ur_description/meshes/ur2/2_upperarm_limb.STL" />
-      </geometry>
-    </collision>
-  </link>
-    <joint name="${ur_prefix}_arm_1_joint" type="revolute"><!-- gazebo has a problem with joint limits where lower limit > higher limit (it internally swaps them around). That's why it's limits under -PI. If I chose 2.5..0.73 as limit, gazebo would only let me move the joints within 0.73..2.5. For now, keep it at -3.943..0.81 and publish joint angles NOT between -PI and PI for this joint (otherwise moveit! would recognise e.g. 3. as illegal, although it's legal).-->
-     <xacro:default_damping_medium/>
-    <xacro:arm_1_limits l="-3.943" u="0.81"/>
-    <origin xyz="0 0.1225 0" rpy="${M_PI} -${M_PI_2} 0" />
-        <parent link="${ur_prefix}_1_shoulder_limb" />
-        <child link="${ur_prefix}_2_upperarm_limb" />
-    <axis xyz="0 0 1" />
-  </joint>
-  <!-- ...........................        -->
-  <link name="${ur_prefix}_ring_3">
-    <inertial>
-      <origin xyz="0 0 0" rpy="0 0 0" />
-      <xacro:cyl_inertia mass="${0.00872/mass_divider}" h="0.02" r="0.04"/>
-    </inertial>
-    <visual>
-      <origin xyz="0.001 0 0" rpy="0 0 0" />
-      <geometry>
-        <mesh filename="package://ur_description/meshes/ur2/ring_3.STL" />
-      </geometry>
-      <material name="">
-        <color rgba="0.5 0.5 0.5 1" />
-      </material>
-    </visual>
-    <collision>
-      <origin xyz="0.001 0 0" rpy="0 0 0" />
-      <geometry>
-        <mesh filename="package://ur_description/meshes/ur2/ring_3.STL" />
-      </geometry>
-    </collision>
-  </link>
-    <joint name="${ur_prefix}_ring_3_joint" type="fixed">
-    <origin xyz="0.41 0 0" rpy="${M_PI} 0 -${M_PI}" />
-        <parent link="${ur_prefix}_2_upperarm_limb" />
-        <child link="${ur_prefix}_ring_3"/>
-    <axis xyz="0 0 0"/>
-  </joint>
-  <!-- ........................... -->
+    <joint name="${ur_prefix}_arm_0_joint" type="revolute">
+      <parent link="${ur_prefix}_0_baseB_limb" />
+      <child link = "${ur_prefix}_1_shoulder_limb" />
+      <origin xyz="0.0 0.0 ${shoulder_height}" rpy="0.0 0.0 0.0" />
+      <axis xyz="0 0 1" />
+      <limit lower="${-2.0 * pi}" upper="${2.0 * pi}" effort="150.0" velocity="3.15"/>
+      <dynamics damping="0.0" friction="0.0"/>
+    </joint>
+    <link name="${ur_prefix}_1_shoulder_limb">
+      <visual>
+        <geometry>
+          <mesh filename="package://ur_description/meshes/ur/shoulder.stl" />
+        </geometry>
+        <material name="LightGrey">
+          <color rgba="0.7 0.7 0.7 1.0"/>
+        </material>
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