Commit message: added world with contact_without_collision objects

File: ur_arm/ur_description/urdf/ur.urdf.xacro (robot description, xacro)
@@ -27,8 +27,8 @@
   </xacro:macro>
   <xacro:macro name="arm_0_limits">
-    <limit effort="8" velocity="1.0" />
+    <limit effort="80" velocity="1.0" />
   </xacro:macro>
   <xacro:macro name="arm_1_limits" params="l u">
-    <limit lower="${l}" upper="${u}" effort="8" velocity="1.0" />
+    <limit lower="${l}" upper="${u}" effort="80" velocity="1.0" />
   </xacro:macro>
     <xacro:macro name="arm_2_limits" params="l u">
@@ -36,11 +36,11 @@
   </xacro:macro>
   <xacro:macro name="arm_3_limits">
-    <limit effort="1.5" velocity="1.0" />
+    <limit effort="10.5" velocity="1.0" />
   </xacro:macro>
   <xacro:macro name="arm_4_limits">
-    <limit effort="1.0" velocity="1.0" />
+    <limit effort="10.0" velocity="1.0" />
   </xacro:macro>
     <xacro:macro name="arm_5_limits">
-    <limit effort="1.0" velocity="1.0" />
+    <limit effort="10.0" velocity="1.0" />
   </xacro:macro>
   <!--- remark 2014: damping greater than 0.5 lead to model break downs when testing it bit by bit -->
@@ -121,28 +121,4 @@
   <gazebo reference="${ur_prefix}base">
     <material>Gazebo/White</material>
-    <xacro:default_material/>
-  </gazebo>
-  <gazebo reference="${ur_prefix}_1_shoulder_limb">
-    <material>Gazebo/FlatBlack</material>
-    <xacro:default_material/>
-  </gazebo>
-  <gazebo reference="${ur_prefix}_2_upperarm_limb">
-    <material>Gazebo/FlatBlack</material>
-    <xacro:default_material/>
-  </gazebo>
-  <gazebo reference="${ur_prefix}_3_forearm_limb">
-    <material>Gazebo/FlatBlack</material>
-    <xacro:default_material/>
-  </gazebo>
-  <gazebo reference="${ur_prefix}_4_upperwrist_limb">
-    <material>Gazebo/FlatBlack</material>
-    <xacro:default_material/>
-  </gazebo>
-  <gazebo reference="${ur_prefix}_5_lowerwrist_limb">
-    <material>Gazebo/FlatBlack</material>
-    <xacro:default_material/>
-  </gazebo>
-  <gazebo reference="${ur_prefix}_6_hand_limb">
-    <material>Gazebo/FlatBlack</material>
     <xacro:default_material/>
   </gazebo>
@@ -282,5 +258,5 @@
       <origin xyz="0.0 0.0 ${shoulder_height}" rpy="0.0 0.0 0.0" />
       <axis xyz="0 0 1" />
-      <limit lower="${-2.0 * pi}" upper="${2.0 * pi}" effort="150.0" velocity="3.15"/>
+      <limit lower="${-2.0 * pi}" upper="${2.0 * pi}" effort="1500.0" velocity="3.15"/>
       <dynamics damping="0.0" friction="0.0"/>
     </joint>
@@ -288,5 +264,5 @@
       <visual>
         <geometry>
-          <mesh filename="package://ur_description/meshes/ur/shoulder.stl" />
+          <mesh filename="package://ur_description/meshes/ur/shoulder.dae" />
         </geometry>
         <material name="LightGrey">
@@ -308,5 +284,5 @@
       <origin xyz="0.0 ${shoulder_offset} 0.0" rpy="0.0 ${pi / 2.0} 0.0" />
       <axis xyz="0 1 0" />
-      <limit lower="${-2.0 * pi}" upper="${2.0 * pi}" effort="150.0" velocity="3.15"/>
+      <limit lower="${-2.0 * pi}" upper="${2.0 * pi}" effort="1500.0" velocity="3.15"/>
       <dynamics damping="0.0" friction="0.0"/>
     </joint>
@@ -314,5 +290,5 @@
       <visual>
         <geometry>
-          <mesh filename="package://ur_description/meshes/ur/upperarm.stl" />
+          <mesh filename="package://ur_description/meshes/ur/upperarm.dae" />
         </geometry>
         <material name="LightGrey">
@@ -340,14 +316,19 @@
       <visual>
         <geometry>
+          <mesh filename="package://ur_description/meshes/ur/forearm.dae" />
+        </geometry>
+        <material name="LightGrey">
+          <color rgba="0.7 0.7 0.7 1.0"/>
+        </material>
+      </visual>
+      <collision>
+        <geometry>
           <mesh filename="package://ur_description/meshes/ur/forearm.stl" />
         </geometry>
-        <material name="LightGrey">
-          <color rgba="0.7 0.7 0.7 1.0"/>
-        </material>
-      </visual>
-      <collision>
-        <geometry>
-          <mesh filename="package://ur_description/meshes/ur/forearm.stl" />
-        </geometry>
+              <surface>
+        <contact>
+          <collide_without_contact>true</collide_without_contact>
+        </contact>
+      </surface>
       </collision>
       <xacro:cylinder_inertial radius="0.06" length="0.5" mass="${forearm_mass}">
@@ -360,5 +341,5 @@
       <origin xyz="0.0 0.0 ${forearm_length}" rpy="0.0 ${pi / 2.0} 0.0" />
       <axis xyz="0 1 0" />
-      <limit lower="${-2.0 * pi}" upper="${2.0 * pi}" effort="28.0" velocity="3.2"/>
+      <limit lower="${-2.0 * pi}" upper="${2.0 * pi}" effort="280.0" velocity="3.2"/>
       <dynamics damping="0.0" friction="0.0"/>
     </joint>
@@ -366,14 +347,19 @@
       <visual>
         <geometry>
+          <mesh filename="package://ur_description/meshes/ur/wrist1.dae" />
+        </geometry>
+        <material name="LightGrey">
+          <color rgba="0.7 0.7 0.7 1.0"/>
+        </material>
+      </visual>
+      <collision>
+        <geometry>
           <mesh filename="package://ur_description/meshes/ur/wrist1.stl" />
         </geometry>
-        <material name="LightGrey">
-          <color rgba="0.7 0.7 0.7 1.0"/>
-        </material>
-      </visual>
-      <collision>
-        <geometry>
-          <mesh filename="package://ur_description/meshes/ur/wrist1.stl" />
-        </geometry>
+              <surface>
+        <contact>
+          <collide_without_contact>true</collide_without_contact>
+        </contact>
+      </surface>
       </collision>
       <xacro:cylinder_inertial radius="0.6" length="0.12" mass="${wrist_1_mass}">
@@ -386,5 +372,5 @@
       <origin xyz="0.0 ${wrist_1_length} 0.0" rpy="0.0 0.0 0.0" />
       <axis xyz="0 0 1" />
-      <limit lower="${-2.0 * pi}" upper="${2.0 * pi}" effort="28.0" velocity="3.2"/>
+      <limit lower="${-2.0 * pi}" upper="${2.0 * pi}" effort="280.0" velocity="3.2"/>
       <dynamics damping="0.0" friction="0.0"/>
     </joint>
@@ -392,14 +378,19 @@
       <visual>
         <geometry>
+          <mesh filename="package://ur_description/meshes/ur/wrist2.dae" />
+        </geometry>
+        <material name="LightGrey">
+          <color rgba="0.7 0.7 0.7 1.0"/>
+        </material>
+      </visual>
+      <collision>
+        <geometry>
           <mesh filename="package://ur_description/meshes/ur/wrist2.stl" />
         </geometry>
-        <material name="LightGrey">
-          <color rgba="0.7 0.7 0.7 1.0"/>
-        </material>
-      </visual>
-      <collision>
-        <geometry>
-          <mesh filename="package://ur_description/meshes/ur/wrist2.stl" />
-        </geometry>
+              <surface>
+        <contact>
+          <collide_without_contact>true</collide_without_contact>
+        </contact>
+      </surface>
       </collision>
       <xacro:cylinder_inertial radius="0.6" length="0.12" mass="${wrist_2_mass}">
@@ -412,5 +403,5 @@
       <origin xyz="0.0 0.0 ${wrist_2_length}" rpy="0.0 0.0 0.0" />
       <axis xyz="0 1 0" />
-      <limit lower="${-2.0 * pi}" upper="${2.0 * pi}" effort="28.0" velocity="3.2"/>
+      <limit lower="${-2.0 * pi}" upper="${2.0 * pi}" effort="280.0" velocity="3.2"/>
       <dynamics damping="0.0" friction="0.0"/>
     </joint>
@@ -418,14 +409,19 @@
       <visual>
         <geometry>
+          <mesh filename="package://ur_description/meshes/ur/wrist3.dae" />
+        </geometry>
+        <material name="LightGrey">
+          <color rgba="0.2 0.2 0.2 1.0"/>
+        </material>
+      </visual>
+      <collision>
+        <geometry>
           <mesh filename="package://ur_description/meshes/ur/wrist3.stl" />
         </geometry>
-        <material name="LightGrey">
-          <color rgba="0.2 0.2 0.2 1.0"/>
-        </material>
-      </visual>
-      <collision>
-        <geometry>
-          <mesh filename="package://ur_description/meshes/ur/wrist3.stl" />
-        </geometry>
+        <surface>
+        <contact>
+          <collide_without_contact>true</collide_without_contact>
+        </contact>
+        </surface>
       </collision>
       <xacro:cylinder_inertial radius="0.6" length="0.12" mass="${wrist_3_mass}">
@@ -463,10 +459,4 @@
     </joint>
     <link name="${ur_prefix}_ee_0_link">
-      <collision>
-        <geometry>
-          <box size="0.01 0.01 0.01"/>
-        </geometry>
-        <origin rpy="0 0 0" xyz="-0.01 0 0"/>
-      </collision>
       <xacro:cylinder_inertial radius="0.06" length="0.012" mass="${wrist_1_mass}">
         <origin xyz="0.0 0.0 0.0" rpy="0 0 0" />
@@ -479,10 +469,4 @@
     </joint>
     <link name="${ur_prefix}_ee_1_link">
-      <collision>
-        <geometry>
-          <box size="0.01 0.01 0.01"/>
-        </geometry>
-        <origin rpy="0 0 0" xyz="-0.01 0 0"/>
-      </collision>
       <xacro:cylinder_inertial radius="0.06" length="0.012" mass="${wrist_1_mass}">
         <origin xyz="0.0 0.0 0.0" rpy="0 0 0" />
@@ -495,10 +479,4 @@
     </joint>
     <link name="${ur_prefix}_ee_2_link">
-      <collision>
-        <geometry>
-          <box size="0.01 0.01 0.01"/>
-        </geometry>
-        <origin rpy="0 0 0" xyz="-0.01 0 0"/>
-      </collision>
       <xacro:cylinder_inertial radius="0.06" length="0.012" mass="${wrist_1_mass}">
         <origin xyz="0.0 0.0 0.0" rpy="0 0 0" />

Commit message: changed the robot's placement to make it coherent with my matlab simulator

File: ur_arm/ur_description/urdf/ur.urdf.xacro (robot description, xacro)
@@ -222,5 +222,5 @@
       <origin xyz="0 0 0" rpy="0 0 0" />
       <geometry>
-        <mesh filename="package://ur_description/meshes/ur/base.stl"/>
+        <mesh filename="package://ur_description/meshes/ur/base.stl" scale="0.001 0.001 0.001"/>
       </geometry>
     </collision>
@@ -243,5 +243,5 @@
       <origin xyz="0 0 0" rpy="0 0 0" />
       <geometry>
-        <mesh filename="package://ur_description/meshes/ur/base.stl" />
+        <mesh filename="package://ur_description/meshes/ur/base.stl" scale="0.001 0.001 0.001"/>
       </geometry>
     </collision>
@@ -258,5 +258,5 @@
       <origin xyz="0.0 0.0 ${shoulder_height}" rpy="0.0 0.0 0.0" />
       <axis xyz="0 0 1" />
-      <limit lower="${-2.0 * pi}" upper="${2.0 * pi}" effort="1500.0" velocity="3.15"/>
+      <limit lower="${-20.0 * pi}" upper="${20.0 * pi}" effort="1500.0" velocity="3.15"/>
       <dynamics damping="0.0" friction="0.0"/>
     </joint>
@@ -272,5 +272,5 @@
       <collision>
         <geometry>
-          <mesh filename="package://ur_description/meshes/ur/shoulder.stl" />
+          <mesh filename="package://ur_description/meshes/ur/shoulder.stl" scale="0.001 0.001 0.001"/>
         </geometry>
       </collision>
@@ -284,5 +284,5 @@
       <origin xyz="0.0 ${shoulder_offset} 0.0" rpy="0.0 ${pi / 2.0} 0.0" />
       <axis xyz="0 1 0" />
-      <limit lower="${-2.0 * pi}" upper="${2.0 * pi}" effort="1500.0" velocity="3.15"/>
+      <limit lower="${-20.0 * pi}" upper="${20.0 * pi}" effort="1500.0" velocity="3.15"/>
       <dynamics damping="0.0" friction="0.0"/>
     </joint>
@@ -298,5 +298,5 @@
       <collision>
         <geometry>
-          <mesh filename="package://ur_description/meshes/ur/upperarm.stl" />
+          <mesh filename="package://ur_description/meshes/ur/upperarm.stl" scale="0.001 0.001 0.001"/>
         </geometry>
       </collision>
@@ -310,5 +310,5 @@
       <origin xyz="0.0 ${elbow_offset} ${upper_arm_length}" rpy="0.0 0.0 0.0" />
       <axis xyz="0 1 0" />
-      <limit lower="${-2.0 * pi}" upper="${2.0 * pi}" effort="150.0" velocity="3.15"/>
+      <limit lower="${-20.0 * pi}" upper="${20.0 * pi}" effort="150.0" velocity="3.15"/>
       <dynamics damping="0.0" friction="0.0"/>
     </joint>
@@ -324,5 +324,5 @@
       <collision>
         <geometry>
-          <mesh filename="package://ur_description/meshes/ur/forearm.stl" />
+          <mesh filename="package://ur_description/meshes/ur/forearm.stl" scale="0.001 0.001 0.001"/>
         </geometry>
               <surface>
@@ -341,5 +341,5 @@
       <origin xyz="0.0 0.0 ${forearm_length}" rpy="0.0 ${pi / 2.0} 0.0" />
       <axis xyz="0 1 0" />
-      <limit lower="${-2.0 * pi}" upper="${2.0 * pi}" effort="280.0" velocity="3.2"/>
+      <limit lower="${-20.0 * pi}" upper="${20.0 * pi}" effort="280.0" velocity="3.2"/>
       <dynamics damping="0.0" friction="0.0"/>
     </joint>
@@ -355,5 +355,5 @@
       <collision>
         <geometry>
-          <mesh filename="package://ur_description/meshes/ur/wrist1.stl" />
+          <mesh filename="package://ur_description/meshes/ur/wrist1.stl" scale="0.001 0.001 0.001"/>
         </geometry>
               <surface>
@@ -372,5 +372,5 @@
       <origin xyz="0.0 ${wrist_1_length} 0.0" rpy="0.0 0.0 0.0" />
       <axis xyz="0 0 1" />
-      <limit lower="${-2.0 * pi}" upper="${2.0 * pi}" effort="280.0" velocity="3.2"/>
+      <limit lower="${-20.0 * pi}" upper="${20.0 * pi}" effort="280.0" velocity="3.2"/>
       <dynamics damping="0.0" friction="0.0"/>
     </joint>
@@ -386,5 +386,5 @@
       <collision>
         <geometry>
-          <mesh filename="package://ur_description/meshes/ur/wrist2.stl" />
+          <mesh filename="package://ur_description/meshes/ur/wrist2.stl" scale="0.001 0.001 0.001"/>
         </geometry>
               <surface>
@@ -403,5 +403,5 @@
       <origin xyz="0.0 0.0 ${wrist_2_length}" rpy="0.0 0.0 0.0" />
       <axis xyz="0 1 0" />
-      <limit lower="${-2.0 * pi}" upper="${2.0 * pi}" effort="280.0" velocity="3.2"/>
+      <limit lower="${-20.0 * pi}" upper="${20.0 * pi}" effort="280.0" velocity="3.2"/>
       <dynamics damping="0.0" friction="0.0"/>
     </joint>
@@ -417,5 +417,5 @@
       <collision>
         <geometry>
-          <mesh filename="package://ur_description/meshes/ur/wrist3.stl" />
+          <mesh filename="package://ur_description/meshes/ur/wrist3.stl" scale="0.001 0.001 0.001"/>
         </geometry>
         <surface>
@@ -434,5 +434,5 @@
       <origin xyz="0.0 0.0 ${wrist_2_length}" rpy="0.0 0.0 0.0" />
       <axis xyz="0 1 0" />
-      <limit lower="${-2.0 * pi}" upper="${2.0 * pi}" effort="0.01" velocity="3.2"/>
+      <limit lower="${-20.0 * pi}" upper="${20.0 * pi}" effort="0.01" velocity="3.2"/>
       <dynamics damping="0.0" friction="0.0"/>
     </joint>
@@ -442,5 +442,5 @@
       <origin xyz="0.0 0.0 ${wrist_2_length}" rpy="0.0 0.0 0.0" />
       <axis xyz="0 1 0" />
-      <limit lower="${-2.0 * pi}" upper="${2.0 * pi}" effort="0.01" velocity="3.2"/>
+      <limit lower="${-20.0 * pi}" upper="${20.0 * pi}" effort="0.01" velocity="3.2"/>
       <dynamics damping="0.0" friction="0.0"/>
     </joint>
@@ -450,5 +450,5 @@
       <origin xyz="0.0 0.0 ${wrist_2_length}" rpy="0.0 0.0 0.0" />
       <axis xyz="0 1 0" />
-      <limit lower="${-2.0 * pi}" upper="${2.0 * pi}" effort="0.01" velocity="3.2"/>
+      <limit lower="${-20.0 * pi}" upper="${20.0 * pi}" effort="0.01" velocity="3.2"/>
       <dynamics damping="0.0" friction="0.0"/>
     </joint>

File: ur_tutorial/ur_on_table/urdf/ur_on_table.urdf.xacro (robot description, xacro)
@@ -21,5 +21,5 @@
 	<xacro:include filename="$(find ur_on_table)/urdf/objects/table.xacro" />
 	<joint name="table_to_arm" type="fixed">
-		<origin xyz="0.40488474042 0.27988474042 0.3" rpy="0 0 -0.785398163397458" />
+		<origin xyz="-0.397270 0.222882 0.3" rpy="0 0 -0.785398163397458" />
 		<parent link="robot_base"/>
 		<child link="table_base"/>
@@ -28,5 +28,5 @@
     <xacro:arm_stand_link link_name="arm_stand"/>
 	<joint name="j2b" type="fixed">
-		<origin xyz="0 -0.035 0" rpy="-1.57079632679 -3.14159265358979 0" /> <!-- set the arm "inside" the table for now because of the rim along the real table. creating a bit of a buffer zone so moveit trajectories are within safe distance of the table edges. -->
+		<origin xyz="0 0 0" rpy="-1.57079632679 -3.14159265358979 -1.57079632679" /> <!-- set the arm "inside" the table for now because of the rim along the real table. creating a bit of a buffer zone so moveit trajectories are within safe distance of the table edges. -->
 		<parent link="tabletop_corner" />
 		<child link="arm_stand" />
@@ -43,5 +43,5 @@
     <xacro:if value="$(arg sensor_on_table)">
         <joint name="toxtion_base" type="fixed">
-            <origin xyz="0 -0.89 -0.01" rpy="0 0 -1.57079632679" />
+            <origin xyz="0 -0.89 -0.01" rpy="0 0 0" />
             <parent link="tabletop_corner" />
             <child link="xtion_base" />

File: ur_tutorial/ur_on_table/urdf/ur_on_table_robot.urdf (robot description, URDF)
Before this commit: robot UrOnTable, 31 links, 30 joints
Links:
- link ur_6_hand_limb: geometry collision mesh filename=package://ur_description/meshes/ur2/6_hand_limb.STL scale=0.001 0.001 0.001; visual mesh filename=package://ur_description/meshes/ur2/6_hand_limb.STL scale=1.0 1.0 1.0

Commit message: small changes

File: ur_arm/ur_description/urdf/ur.urdf.xacro (robot description, xacro)
@@ -222,5 +222,5 @@
       <origin xyz="0 0 0" rpy="0 0 0" />
       <geometry>
-        <mesh filename="package://ur_description/meshes/ur/base.stl" scale="0.001 0.001 0.001"/>
+        <mesh filename="package://ur_description/meshes/ur/base.stl" scale="1 1 1"/>
       </geometry>
     </collision>
@@ -243,5 +243,5 @@
       <origin xyz="0 0 0" rpy="0 0 0" />
       <geometry>
-        <mesh filename="package://ur_description/meshes/ur/base.stl" scale="0.001 0.001 0.001"/>
+        <mesh filename="package://ur_description/meshes/ur/base.stl" scale="1 1 1"/>
       </geometry>
     </collision>
@@ -272,5 +272,5 @@
       <collision>
         <geometry>
-          <mesh filename="package://ur_description/meshes/ur/shoulder.stl" scale="0.001 0.001 0.001"/>
+          <mesh filename="package://ur_description/meshes/ur/shoulder.stl" scale="1 1 1"/>
         </geometry>
       </collision>
@@ -298,5 +298,5 @@
       <collision>
         <geometry>
-          <mesh filename="package://ur_description/meshes/ur/upperarm.stl" scale="0.001 0.001 0.001"/>
+          <mesh filename="package://ur_description/meshes/ur/upperarm.stl" scale="1 1 1"/>
         </geometry>
       </collision>
@@ -324,5 +324,5 @@
       <collision>
         <geometry>
-          <mesh filename="package://ur_description/meshes/ur/forearm.stl" scale="0.001 0.001 0.001"/>
+          <mesh filename="package://ur_description/meshes/ur/forearm.stl" scale="1 1 1"/>
         </geometry>
               <surface>
@@ -355,5 +355,5 @@
       <collision>
         <geometry>
-          <mesh filename="package://ur_description/meshes/ur/wrist1.stl" scale="0.001 0.001 0.001"/>
+          <mesh filename="package://ur_description/meshes/ur/wrist1.stl" scale="1 1 1"/>
         </geometry>
               <surface>
@@ -386,5 +386,5 @@
       <collision>
         <geometry>
-          <mesh filename="package://ur_description/meshes/ur/wrist2.stl" scale="0.001 0.001 0.001"/>
+          <mesh filename="package://ur_description/meshes/ur/wrist2.stl" scale="1 1 1"/>
         </geometry>
               <surface>
@@ -417,5 +417,5 @@
       <collision>
         <geometry>
-          <mesh filename="package://ur_description/meshes/ur/wrist3.stl" scale="0.001 0.001 0.001"/>
+          <mesh filename="package://ur_description/meshes/ur/wrist3.stl" scale="1 1 1"/>
         </geometry>
         <surface>

Commit message: ajout de l'adater dans le robot

File: ur_arm/ur_description/urdf/ur.urdf.xacro (robot description, xacro)
@@ -429,4 +429,19 @@
       </xacro:cylinder_inertial>
     </link>
+    <joint name="${ur_prefix}_adapter_fixed_joint" type="fixed">
+      <parent link="${ur_prefix}_6_hand_limb" />
+      <child link = "${ur_prefix}_adapter_link" />
+      <origin xyz="-0.0375 ${wrist_3_length} -0.0375" rpy="0.0 0.0 0" />
+    </joint>
+    <link name="${ur_prefix}_adapter_link">
+    <visual>
+        <geometry>
+              <mesh filename="package://ur_description/meshes/ur/adapter.STL" scale="0.001 0.001 0.001"/>
+        </geometry>
+    </visual>
+      <xacro:cylinder_inertial radius="0.06" length="0.012" mass="${wrist_1_mass}">
+        <origin xyz="0.0 0.0 0.0" rpy="0 0 0" />
+      </xacro:cylinder_inertial>
+    </link>
     <joint name="${ur_prefix}_finger_joint_0" type="revolute">
       <parent link="${ur_prefix}_ee_link" />

Commit message: dae added to gazebo

File: ur_arm/ur_description/urdf/ur.urdf.xacro (robot description, xacro)
@@ -437,5 +437,5 @@
     <visual>
         <geometry>
-              <mesh filename="package://ur_description/meshes/ur/adapter.STL" scale="0.001 0.001 0.001"/>
+              <mesh filename="package://ur_description/meshes/ur/adapter.dae" scale="0.001 0.001 0.001"/>
         </geometry>
     </visual>
