Commit message: try pour remove la limite angulaire

File: ur_tutorial/ur_on_table/urdf/ur_on_table_robot.urdf (robot description, URDF)
Before this commit: robot UrOnTable, 31 links, 30 joints
Joints:
- joint ur_arm_1_joint: limit lower=-3.943 upper=0.81 effort=8 velocity=1.0 -> effort=8 velocity=1.0
- joint ur_arm_2_joint: limit lower=-4.395 upper=1.252 effort=4 velocity=1.0 -> effort=4 velocity=1.0
